Commit message: Add files via upload

File: rover_description/urdf/rover.xacro (robot description, xacro)
@@ -4,4 +4,7 @@
   <xacro:property name="cameraMass" value="0.1" />
   <xacro:include filename="$(find rover_description)/urdf/rover.gazebo" />
+  <xacro:include filename="$(find rover_description)/urdf/materials.xacro" />
+  <!--adding
+  colur to the robot in gazebo this will not visualized in rviz -->
   <gazebo reference="base_body">
     <material>Gazebo/Red</material>
@@ -21,19 +24,7 @@
   <!-- Base base_footprint -->
   <link name="base_body">
-    <collision>
-      <origin xyz="0.1 0 1.5" rpy="0 0 0" />
-      <geometry>
-        <mesh filename="package://rover_description/meshes/Bot_Body.stl" />
-      </geometry>
-    </collision>
-    <visual name='base_body_visual'>
-      <origin xyz="0.1 0 1.8" rpy="0 0 0" />
-      <geometry>
-        <mesh filename="package://rover_description/meshes/Bot_Body.stl" />
-      </geometry>
-    </visual>
-    <inertial>
-      <origin xyz="0 0 1" rpy="0 0 0" />
-      <mass value="0.1" />
+    <inertial>
+      <origin xyz="0 0 0.54" rpy="0 0 0" />
+      <mass value="1" />
       <inertia
         ixx="0.001" ixy="0.0" ixz="0.0"
@@ -41,30 +32,94 @@
         izz="0.001" />
     </inertial>
-  </link>
+    <collision>
+      <origin xyz="0 0 0.54" rpy="0 0 0" />
+      <geometry>
+        <mesh filename="package://rover_description/meshes/Bot_Body.stl" scale="0.3 0.3 0.3" />
+      </geometry>
+    </collision>
+    <visual name='base_body_visual'>
+      <origin xyz="0 0 0.54" rpy="0 0 0" />
+      <geometry>
+        <mesh filename="package://rover_description/meshes/Bot_Body.stl" scale="0.3 0.3 0.3" />
+      </geometry>
+    </visual>
+  </link>
+  <!-- Create wheel right -->
+  <link name="right_wheel">
+    <inertial>
+      <mass value="0.2" />
+      <origin rpy="${pi} ${pi/2} 0" xyz="0 0 0" />
+      <inertia ixx="0.00052666666" ixy="0" ixz="0" iyy="0.00052666666" iyz="0" izz="0.001" />
+    </inertial>
+    <collision name="link_right_wheel_collision">
+      <origin rpy="${pi} ${pi/2} 0" xyz="0 0 0" />
+      <geometry>
+        <mesh filename="package://rover_description/meshes/Wheel.STL" scale="1.25 1.25 1.25" />
+      </geometry>
+    </collision>
+    <visual>
+      <origin rpy="${pi} ${pi/2} 0" xyz="0 0 0" />
+      <geometry>
+        <mesh filename="package://rover_description/meshes/Wheel.STL" scale="1.25 1.25 1.25" />
+      </geometry>
+      <!-- <material name="black" /> -->
+    </visual>
+  </link>
+  <joint name="right_wheel_joint" type="continuous">
+    <parent link="base_body" />
+    <child link="right_wheel" />
+    <origin rpy="0 0 ${pi}" xyz="0.43 0.3 0.25" />
+    <limit effort="10000" velocity="1000" />
+    <joint_properties damping="1.0" friction="1.0" />
+  </joint>
+  <!-- Create wheel left -->
+  <link name="left_wheel">
+    <inertial>
+      <mass value="0.2" />
+      <origin rpy="0 ${pi} 0" xyz="0 0 0" />
+      <inertia ixx="0.00052666666" ixy="0" ixz="0" iyy="0.00052666666" iyz="0" izz="0.001" />
+    </inertial>
+    <collision name="link_left_wheel_collision">
+      <origin rpy="0 ${pi/2} 0" xyz="0 0 0" />
+      <geometry>
+        <mesh filename="package://rover_description/meshes/Wheel.STL" scale="1.25 1.25 1.25" />
+      </geometry>
+    </collision>
+    <visual>
+      <origin rpy="0 ${pi/2} 0" xyz="0 0 0" />
+      <geometry>
+        <mesh filename="package://rover_description/meshes/Wheel.STL" scale="1.25 1.25 1.25" />
+      </geometry>
+      <!-- <material name="black" /> -->
+    </visual>
+  </link>
+  <joint name="left_wheel_joint" type="continuous">
+    <parent link="base_body" />
+    <child link="left_wheel" />
+    <origin rpy="0 0 ${pi}" xyz="-0.43 0.3 0.25" />
+    <limit effort="10000" velocity="1000" />
+    <joint_properties damping="1.0" friction="1.0" />
+  </joint>
   <!--Castor
-  Plate  -->
+  wheel Plate  -->
   <link name="caster_plate_link">
     <visual>
-      <origin rpy="1.57079632679 0 0" xyz="0 -1.85 0.8" />
-      <geometry>
-        <mesh filename="package://rover_description/meshes/Bot_Castor_Plate.stl" />
-      </geometry>
-    </visual>
-    <collision>
-      <geometry>
-        <mesh filename="package://rover_description/meshes/Bot_Castor_Plate.stl" />
-      </geometry>
-      <origin rpy="1.57079632679 0 0" xyz="0 -1.85 0.8" />
-    </collision>
-    <inertial>
-      <mass value="0.2" />
-      <origin xyz="0 0 0" />
-      <inertia ixx="0.001" ixy="0.0" ixz="0.0" iyy="0.001" iyz="0.0" izz="0.001" />
-    </inertial>
+      <origin rpy="0 0 0" xyz="0 0 0" />
+      <geometry>
+        <mesh filename="package://rover_description/meshes/Bot_Castor_Plate.stl" scale="0.3 0.3 0.3" />
+      </geometry>
+      <material name="black" />
+    </visual>
+    <collision>
+      <geometry>
+        <mesh filename="package://rover_description/meshes/Bot_Castor_Plate.stl" scale="0.3 0.3 0.3" />
+      </geometry>
+      <origin rpy="0 0 0" xyz="0 0 0" />
+    </collision>
   </link>
   <joint name="caster_plate_joint" type="fixed">
     <parent link="base_body" />
     <child link="caster_plate_link" />
-    <origin rpy="-1.57079632679 0 0" xyz="0 1 0" />
+    <origin rpy="0 0 0" xyz="0 0 0.56" />
   </joint>
   <!--Caster
@@ -72,30 +127,36 @@
   <link name="caster_wheel_link">
     <visual>
-      <origin rpy="1.57079632679 0 0" xyz="0 -1.85 0.8" />
-      <geometry>
-        <mesh filename="package://rover_description/meshes/Bot_Castor_Wheel.stl" />
-      </geometry>
-    </visual>
-    <collision>
-      <geometry>
-        <mesh filename="package://rover_description/meshes/Bot_Castor_Wheel.stl" />
-      </geometry>
-      <origin rpy="1.57079632679 0 0" xyz="0 -1.85 0.8" />
-    </collision>
-    <inertial>
-      <mass value="0.2" />
-      <origin xyz="0 0 0" />
-      <inertia ixx="0.001" ixy="0.0" ixz="0.0" iyy="0.001" iyz="0.0" izz="0.001" />
-    </inertial>
+      <origin rpy="0 0 0" xyz="0 0 0" />
+      <geometry>
+        <mesh filename="package://rover_description/meshes/Bot_Castor_Wheel.stl" scale="0.3 0.3 0.3" />
+      </geometry>
+      <material name="black" />
+    </visual>
+    <collision>
+      <geometry>
+        <mesh filename="package://rover_description/meshes/Bot_Castor_Wheel.stl" scale="0.3 0.3 0.3" />
+      </geometry>
+      <origin rpy="0 0 0" xyz="0 0 0" />
+    </collision>
+    <surface>
+      <friction>
+        <ode>
+          <mu>0</mu>
+          <mu2>0</mu2>
+          <slip1>1.0</slip1>
+          <slip2>1.0</slip2>
+        </ode>
+      </friction>
+    </surface>
   </link>
   <joint name="caster_front_joint" type="fixed">
     <parent link="base_body" />
     <child link="caster_wheel_link" />
-    <origin rpy="-1.57079632679 0 0" xyz="0 1 0" />
-  </joint>
-   <!-- Hokuyo Laser -->
+    <origin rpy="0 0 0" xyz="0 0 0.56" />
+  </joint>
+  <!-- Hokuyo Laser -->
   <joint name="hokuyo_joint" type="fixed">
     <axis xyz="0 1 0" />
-    <origin xyz="0 0.5 2.85" rpy="0 0 1.57" />
+    <origin xyz="0 0.15 0.88" rpy="0 0 ${pi/2}" />
     <parent link="base_body" />
     <child link="hokuyo" />
@@ -121,17 +182,25 @@
   </link>
   <gazebo>
-    <plugin filename="libgazebo_ros_diff_drive.so" name="differential_drive_controller">
-      <legacyMode>false</legacyMode>
+    <plugin name="differential_drive_controller" filename="libgazebo_ros_diff_drive.so">
+      <robotNamespace />
       <alwaysOn>true</alwaysOn>
-      <updateRate>20</updateRate>
-      <leftJoint>joint_left_wheel</leftJoint>
-      <rightJoint>joint_right_wheel</rightJoint>
-      <wheelSeparation>0.2</wheelSeparation>
-      <wheelDiameter>0.2</wheelDiameter>
-      <torque>0.1</torque>
+      <updateRate>10</updateRate>
+      <legacyMode>true</legacyMode>
+      <leftJoint>left_wheel_joint</leftJoint>
+      <rightJoint>right_wheel_joint</rightJoint>
+      <wheelSeparation>0.5380</wheelSeparation>
+      <wheelDiameter>0.2410</wheelDiameter>
+      <torque>20</torque>
       <commandTopic>cmd_vel</commandTopic>
       <odometryTopic>odom</odometryTopic>
       <odometryFrame>odom</odometryFrame>
-      <robotBaseFrame>link_chassis</robotBaseFrame>
+      <robotBaseFrame>base_body</robotBaseFrame>
+      <publishWheelTF>false</publishWheelTF>
+      <publishWheelJointState>false</publishWheelJointState>
+      <rosDebugLevel>na</rosDebugLevel>
+      <wheelAcceleration>0</wheelAcceleration>
+      <wheelTorque>5</wheelTorque>
+      <odometrySource>world</odometrySource>
+      <publishTf>1</publishTf>
     </plugin>
   </gazebo>

Commit message: Add files via upload

File: rover_description/urdf/rover.xacro (robot description, xacro)
@@ -5,6 +5,4 @@
   <xacro:include filename="$(find rover_description)/urdf/rover.gazebo" />
   <xacro:include filename="$(find rover_description)/urdf/materials.xacro" />
-  <!--adding
-  colur to the robot in gazebo this will not visualized in rviz -->
   <gazebo reference="base_body">
     <material>Gazebo/Red</material>
@@ -101,58 +99,69 @@
     <joint_properties damping="1.0" friction="1.0" />
   </joint>
-  <!--Castor
-  wheel Plate  -->
-  <link name="caster_plate_link">
-    <visual>
-      <origin rpy="0 0 0" xyz="0 0 0" />
-      <geometry>
-        <mesh filename="package://rover_description/meshes/Bot_Castor_Plate.stl" scale="0.3 0.3 0.3" />
+   <!-- caster plate -->
+  <link name="caster_plate">
+    <inertial>
+      <mass value="0.2" />
+      <origin rpy="${-pi/2} 0 0" xyz="0 0 0" />
+      <inertia ixx="0.00052666666" ixy="0" ixz="0" iyy="0.00052666666" iyz="0" izz="0.001" />
+    </inertial>
+    <collision name="link_caster_plate_collision">
+      <origin rpy="${-pi/2} 0 0" xyz="0 0 0" />
+      <geometry>
+        <mesh filename="package://rover_description/meshes/caster_part.STL" scale="1 1 1" />
+      </geometry>
+    </collision>
+    <visual>
+      <origin rpy="${-pi/2} 0 0" xyz="0 0 0" />
+      <geometry>
+        <mesh filename="package://rover_description/meshes/caster_part.STL" scale="1 1 1" />
       </geometry>
       <material name="black" />
     </visual>
-    <collision>
-      <geometry>
-        <mesh filename="package://rover_description/meshes/Bot_Castor_Plate.stl" scale="0.3 0.3 0.3" />
-      </geometry>
-      <origin rpy="0 0 0" xyz="0 0 0" />
-    </collision>
-  </link>
-  <joint name="caster_plate_joint" type="fixed">
-    <parent link="base_body" />
-    <child link="caster_plate_link" />
-    <origin rpy="0 0 0" xyz="0 0 0.56" />
-  </joint>
-  <!--Caster
-  wheel  -->
-  <link name="caster_wheel_link">
-    <visual>
-      <origin rpy="0 0 0" xyz="0 0 0" />
-      <geometry>
-        <mesh filename="package://rover_description/meshes/Bot_Castor_Wheel.stl" scale="0.3 0.3 0.3" />
+  </link>
+  <joint name="caster_plate_joint" type="continuous">
+    <parent link="base_body" />
+    <child link="caster_plate" />
+    <origin rpy="0 0 0" xyz="0 -0.3 0.23" />
+    <axis xyz="0 0 1" />
+    <limit effort="10000" velocity="1000" />
+    <joint_properties damping="1.0" friction="1.0" />
+  </joint>
+  <!-- caster wheel -->
+  <link name="caster_wheel">
+    <inertial>
+      <mass value="0.2" />
+      <origin rpy="0 ${pi} 0" xyz="0 0 0" />
+      <inertia ixx="0.00052666666" ixy="0" ixz="0" iyy="0.00052666666" iyz="0" izz="0.001" />
+    </inertial>
+    <collision name="link_left_wheel_collision">
+      <origin rpy="0 ${pi/2} 0" xyz="0 0 0" />
+      <geometry>
+        <mesh filename="package://rover_description/meshes/caster_wheel.STL" scale="1 1 1" />
+      </geometry>
+    </collision>
+    <visual>
+      <origin rpy="0 ${pi/2} 0" xyz="0 0 0" />
+      <geometry>
+        <mesh filename="package://rover_description/meshes/caster_wheel.STL" scale="1 1 1" />
       </geometry>
       <material name="black" />
     </visual>
-    <collision>
-      <geometry>
-        <mesh filename="package://rover_description/meshes/Bot_Castor_Wheel.stl" scale="0.3 0.3 0.3" />
-      </geometry>
-      <origin rpy="0 0 0" xyz="0 0 0" />
-    </collision>
-    <surface>
-      <friction>
-        <ode>
-          <mu>0</mu>
-          <mu2>0</mu2>
-          <slip1>1.0</slip1>
-          <slip2>1.0</slip2>
-        </ode>
-      </friction>
-    </surface>
-  </link>
-  <joint name="caster_front_joint" type="fixed">
-    <parent link="base_body" />
-    <child link="caster_wheel_link" />
-    <origin rpy="0 0 0" xyz="0 0 0.56" />
-  </joint>
+  </link>
+  <joint name="caster_wheel_joint" type="continuous">
+    <parent link="caster_plate" />
+    <child link="caster_wheel" />
+    <origin rpy="0 0 ${pi}" xyz="0 0.05 -0.15" />
+    <limit effort="10000" velocity="1000" />
+    <joint_properties damping="1.0" friction="1.0" />
+  </joint>
+  <gazebo reference="caster_wheel_link">
+    <mu1>0.0</mu1>
+    <mu2>0.0</mu2>
+    <kp>1000000.0</kp>
+    <kd>100.0</kd>
+    <minDepth>0.001</minDepth>
+    <maxVel>1.0</maxVel>
+  </gazebo>
   <!-- Hokuyo Laser -->
   <joint name="hokuyo_joint" type="fixed">
@@ -220,5 +229,5 @@
         </scan>
         <range>
-          <min>0.10</min>
+          <min>0.1</min>
           <max>30.0</max>
           <resolution>0.01</resolution>
@@ -227,5 +236,5 @@
           <type>gaussian</type>
           <mean>0.0</mean>
-          <stddev>0.01</stddev>
+          <stddev>0.0</stddev>
         </noise>
       </ray>
