Commit message: Add files via upload

File: rover_description/urdf/rover.xacro (robot description, xacro)
@@ -14,14 +14,21 @@
     <material>Gazebo/Black</material>
   </gazebo>
-  <gazebo reference="caster_wheel_link">
+  <gazebo reference="caster_wheel">
     <material>Gazebo/Black</material>
   </gazebo>
-  <gazebo reference="caster_plate_link">
+  <gazebo reference="caster_plate">
     <material>Gazebo/Black</material>
   </gazebo>
   <!-- Base base_footprint -->
   <link name="base_body">
-    <inertial>
-      <origin xyz="0 0 0.54" rpy="0 0 0" />
+    <!-- <inertial>
+      <origin xyz="0 0 0.34" rpy="0 0 0" />
+      <mass value="8.2573504e-01" />
+      <inertia ixx="2.2124416e-03" ixy="-1.2294101e-05" ixz="3.4938785e-05"
+        iyy="2.1193702e-03" iyz="-5.0120904e-06"
+        izz="2.0064271e-03" />
+    </inertial> -->
+    <inertial>
+      <origin xyz="0 0 0.34" rpy="0 0 0" />
       <mass value="1" />
       <inertia
@@ -31,13 +38,13 @@
     </inertial>
     <collision>
-      <origin xyz="0 0 0.54" rpy="0 0 0" />
-      <geometry>
-        <mesh filename="package://rover_description/meshes/Bot_Body.stl" scale="0.3 0.3 0.3" />
+      <origin xyz="0 0 0.34" rpy="0 0 0" />
+      <geometry>
+        <mesh filename="package://rover_description/meshes/Bot_Body.stl" scale="0.1 0.1 0.1" />
       </geometry>
     </collision>
     <visual name='base_body_visual'>
-      <origin xyz="0 0 0.54" rpy="0 0 0" />
-      <geometry>
-        <mesh filename="package://rover_description/meshes/Bot_Body.stl" scale="0.3 0.3 0.3" />
+      <origin xyz="0 0 0.34" rpy="0 0 0" />
+      <geometry>
+        <mesh filename="package://rover_description/meshes/Bot_Body.stl" scale="0.1 0.1 0.1" />
       </geometry>
     </visual>
@@ -45,4 +52,11 @@
   <!-- Create wheel right -->
   <link name="right_wheel">
+    <!-- <inertial>
+      <origin rpy="${pi} ${pi/2} 0" xyz="0 0 0" />
+      <mass value="2.8498940e-02" />
+      <inertia ixx="1.1175580e-05" ixy="-4.2369783e-11" ixz="-5.9381719e-09"
+        iyy="1.1192413e-05" iyz="-1.4400107e-11"
+        izz="2.0712558e-05" />
+    </inertial> -->
     <inertial>
       <mass value="0.2" />
@@ -53,5 +67,5 @@
       <origin rpy="${pi} ${pi/2} 0" xyz="0 0 0" />
       <geometry>
-        <mesh filename="package://rover_description/meshes/Wheel.STL" scale="1.25 1.25 1.25" />
+        <mesh filename="package://rover_description/meshes/Wheel.STL" scale="0.4 0.4 0.4" />
       </geometry>
     </collision>
@@ -59,7 +73,7 @@
       <origin rpy="${pi} ${pi/2} 0" xyz="0 0 0" />
       <geometry>
-        <mesh filename="package://rover_description/meshes/Wheel.STL" scale="1.25 1.25 1.25" />
-      </geometry>
-      <!-- <material name="black" /> -->
+        <mesh filename="package://rover_description/meshes/Wheel.STL" scale="0.4 0.4 0.4" />
+      </geometry>
+      <material name="black" />
     </visual>
   </link>
@@ -67,96 +81,30 @@
     <parent link="base_body" />
     <child link="right_wheel" />
-    <origin rpy="0 0 ${pi}" xyz="0.43 0.3 0.25" />
+    <origin rpy="0 0 ${pi}" xyz="0.14 0.10 0.25" />
+    <axis xyz="1 0 0" />
     <limit effort="10000" velocity="1000" />
     <joint_properties damping="1.0" friction="1.0" />
   </joint>
-  <!-- Create wheel left -->
-  <link name="left_wheel">
-    <inertial>
-      <mass value="0.2" />
-      <origin rpy="0 ${pi} 0" xyz="0 0 0" />
-      <inertia ixx="0.00052666666" ixy="0" ixz="0" iyy="0.00052666666" iyz="0" izz="0.001" />
-    </inertial>
-    <collision name="link_left_wheel_collision">
-      <origin rpy="0 ${pi/2} 0" xyz="0 0 0" />
-      <geometry>
-        <mesh filename="package://rover_description/meshes/Wheel.STL" scale="1.25 1.25 1.25" />
-      </geometry>
-    </collision>
-    <visual>
-      <origin rpy="0 ${pi/2} 0" xyz="0 0 0" />
-      <geometry>
-        <mesh filename="package://rover_description/meshes/Wheel.STL" scale="1.25 1.25 1.25" />
-      </geometry>
-      <!-- <material name="black" /> -->
-    </visual>
-  </link>
-  <joint name="left_wheel_joint" type="continuous">
-    <parent link="base_body" />
-    <child link="left_wheel" />
-    <origin rpy="0 0 ${pi}" xyz="-0.43 0.3 0.25" />
-    <limit effort="10000" velocity="1000" />
-    <joint_properties damping="1.0" friction="1.0" />
-  </joint>
-   <!-- caster plate -->
-  <link name="caster_plate">
-    <inertial>
-      <mass value="0.2" />
-      <origin rpy="${-pi/2} 0 0" xyz="0 0 0" />
-      <inertia ixx="0.00052666666" ixy="0" ixz="0" iyy="0.00052666666" iyz="0" izz="0.001" />
-    </inertial>
-    <collision name="link_caster_plate_collision">
-      <origin rpy="${-pi/2} 0 0" xyz="0 0 0" />
-      <geometry>
-        <mesh filename="package://rover_description/meshes/caster_part.STL" scale="1 1 1" />
-      </geometry>
-    </collision>
-    <visual>
-      <origin rpy="${-pi/2} 0 0" xyz="0 0 0" />
-      <geometry>
-        <mesh filename="package://rover_description/meshes/caster_part.STL" scale="1 1 1" />
-      </geometry>
-      <material name="black" />
-    </visual>
-  </link>
-  <joint name="caster_plate_joint" type="continuous">
-    <parent link="base_body" />
-    <child link="caster_plate" />
-    <origin rpy="0 0 0" xyz="0 -0.3 0.23" />
-    <axis xyz="0 0 1" />
-    <limit effort="10000" velocity="1000" />
-    <joint_properties damping="1.0" friction="1.0" />
-  </joint>
-  <!-- caster wheel -->
-  <link name="caster_wheel">
-    <inertial>
-      <mass value="0.2" />
-      <origin rpy="0 ${pi} 0" xyz="0 0 0" />
-      <inertia ixx="0.00052666666" ixy="0" ixz="0" iyy="0.00052666666" iyz="0" izz="0.001" />
-    </inertial>
-    <collision name="link_left_wheel_collision">
-      <origin rpy="0 ${pi/2} 0" xyz="0 0 0" />
-      <geometry>
-        <mesh filename="package://rover_description/meshes/caster_wheel.STL" scale="1 1 1" />
-      </geometry>
-    </collision>
-    <visual>
-      <origin rpy="0 ${pi/2} 0" xyz="0 0 0" />
-      <geometry>
-        <mesh filename="package://rover_description/meshes/caster_wheel.STL" scale="1 1 1" />
-      </geometry>
-      <material name="black" />
-    </visual>
-  </link>
-  <joint name="caster_wheel_joint" type="continuous">
-    <parent link="caster_plate" />
-    <child link="caster_wheel" />
-    <origin rpy="0 0 ${pi}" xyz="0 0.05 -0.15" />
-    <limit effort="10000" velocity="1000" />
-    <joint_properties damping="1.0" friction="1.0" />
-  </joint>
-  <gazebo reference="caster_wheel_link">
-    <mu1>0.0</mu1>
-    <mu2>0.0</mu2>
+  <gazebo reference="right_wheel">
+    <mu1>0.1</mu1>
+    <mu2>0.1</mu2>
+    <kp>500000.0</kp>
+    <kd>10.0</kd>
+    <minDepth>0.001</minDepth>
+    <maxVel>0.1</maxVel>
+    <fdir1>1 0 0</fdir1>
+  </gazebo>
+  <gazebo reference="left_wheel">
+    <mu1>0.1</mu1>
+    <mu2>0.1</mu2>
+    <kp>500000.0</kp>
+    <kd>10.0</kd>
+    <minDepth>0.001</minDepth>
+    <maxVel>0.1</maxVel>
+    <fdir1>1 0 0</fdir1>
+  </gazebo>
+  <gazebo reference="caster_wheel">
+    <mu1>0.1</mu1>
+    <mu2>0.1</mu2>
     <kp>1000000.0</kp>
     <kd>100.0</kd>
@@ -164,8 +112,115 @@
     <maxVel>1.0</maxVel>
   </gazebo>
+  <!-- Create wheel left -->
+  <link name="left_wheel">
+    <!-- <inertial>
+      <origin rpy="0 ${pi/2} 0" xyz="0 0 0" />
+      <mass value="2.8498940e-02" />
+      <inertia ixx="1.1175580e-05" ixy="-4.2369783e-11" ixz="-5.9381719e-09"
+        iyy="1.1192413e-05" iyz="-1.4400107e-11"
+        izz="2.0712558e-05" />
+    </inertial> -->
+    <inertial>
+      <mass value="0.2" />
+      <origin rpy="0 ${pi/2} 0" xyz="0 0 0" />
+      <inertia ixx="0.00052666666" ixy="0" ixz="0" iyy="0.00052666666" iyz="0" izz="0.001" />
+    </inertial>
+    <collision name="link_left_wheel_collision">
+      <origin rpy="0 ${pi/2} 0" xyz="0 0 0" />
+      <geometry>
+        <mesh filename="package://rover_description/meshes/Wheel.STL" scale="0.4 0.4 0.4" />
+      </geometry>
+    </collision>
+    <visual>
+      <origin rpy="0 ${pi/2} 0" xyz="0 0 0" />
+      <geometry>
+        <mesh filename="package://rover_description/meshes/Wheel.STL" scale="0.4 0.4 0.4" />
+      </geometry>
+      <material name="black" />
+    </visual>
+  </link>
+  <joint name="left_wheel_joint" type="continuous">
+    <parent link="base_body" />
+    <child link="left_wheel" />
+    <origin rpy="0 0 ${pi}" xyz="-0.14 0.10 0.25" />
+    <axis xyz="1 0 0" />
+    <limit effort="10000" velocity="1000" />
+    <joint_properties damping="1.0" friction="1.0" />
+  </joint>
+  <!-- caster plate -->
+  <link name="caster_plate">
+    <!-- <inertial>
+      <origin rpy="${-pi/2} 0 0" xyz="0 0 0" />
+      <mass value="0.05" />
+      <inertia ixx="0.1" ixy="0.0" ixz="0.0"
+               iyy="0.1" iyz="0.0"
+               izz="0.01" />
+    </inertial> -->
+    <inertial>
+      <mass value="0.2" />
+      <origin rpy="${-pi/2} 0 0" xyz="0 0 0" />
+      <inertia ixx="0.00052666666" ixy="0" ixz="0" iyy="0.00052666666" iyz="0" izz="0.001" />
+    </inertial>
+    <collision name="link_caster_plate_collision">
+      <origin rpy="${-pi/2} 0 0" xyz="0 0 0" />
+      <geometry>
+        <mesh filename="package://rover_description/meshes/caster_part.STL" scale="0.25 0.25 0.25" />
+      </geometry>
+    </collision>
+    <visual>
+      <origin rpy="${-pi/2} 0 0" xyz="0 0 0" />
+      <geometry>
+        <mesh filename="package://rover_description/meshes/caster_part.STL" scale="0.25 0.25 0.25" />
+      </geometry>
+      <material name="black" />
+    </visual>
+  </link>
+  <joint name="caster_plate_joint" type="continuous">
+    <parent link="base_body" />
+    <child link="caster_plate" />
+    <origin rpy="0 0 0" xyz="0 -0.1 0.24" />
+    <axis xyz="0 0 1" />
+    <limit effort="10000" velocity="1000" />
+    <joint_properties damping="1.0" friction="1.0" />
+  </joint>
+  <!-- caster wheel -->
+  <link name="caster_wheel">
+    <!-- <inertial>
+      <origin rpy="0 ${pi} 0" xyz="0 0 0" />
+      <mass value="0.005" />
+      <inertia ixx="0.01" ixy="0.0" ixz="0.0"
+               iyy="0.01" iyz="0.0"
+               izz="0.01" />
+    </inertial> -->
+    <inertial>
+      <mass value="0.1" />
+      <origin rpy="0 ${pi} 0" xyz="0 0 0" />
+      <inertia ixx="0.00052666666" ixy="0" ixz="0" iyy="0.00052666666" iyz="0" izz="0.001" />
+    </inertial>
+    <collision name="link_left_wheel_collision">
+      <origin rpy="0 ${pi/2} 0" xyz="0 0 0" />
+      <geometry>
+        <mesh filename="package://rover_description/meshes/caster_wheel.STL" scale="0.25 0.25 0.25" />
+      </geometry>
+    </collision>
+    <visual>
+      <origin rpy="0 ${pi/2} 0" xyz="0 0 0" />
+      <geometry>
+        <mesh filename="package://rover_description/meshes/caster_wheel.STL" scale="0.25 0.25 0.25" />
+      </geometry>
+      <material name="black" />
+    </visual>
+  </link>
+  <joint name="caster_wheel_joint" type="continuous">
+    <parent link="caster_plate" />
+    <child link="caster_wheel" />
+    <origin rpy="0 0 ${pi}" xyz="0 0.014 -0.0355" />
+    <limit effort="10000" velocity="1000" />
+    <joint_properties damping="1.0" friction="1.0" />
+  </joint>
   <!-- Hokuyo Laser -->
   <joint name="hokuyo_joint" type="fixed">
     <axis xyz="0 1 0" />
-    <origin xyz="0 0.15 0.88" rpy="0 0 ${pi/2}" />
+    <origin xyz="0 0.05 0.47" rpy="0 0 ${pi/2}" />
     <parent link="base_body" />
     <child link="hokuyo" />
@@ -194,11 +249,11 @@
       <robotNamespace />
       <alwaysOn>true</alwaysOn>
-      <updateRate>10</updateRate>
-      <legacyMode>true</legacyMode>
+      <updateRate>30</updateRate>
+      <legacyMode>false</legacyMode>
       <leftJoint>left_wheel_joint</leftJoint>
       <rightJoint>right_wheel_joint</rightJoint>
-      <wheelSeparation>0.5380</wheelSeparation>
-      <wheelDiameter>0.2410</wheelDiameter>
-      <torque>20</torque>
+      <wheelSeparation>0.5</wheelSeparation>
+      <wheelDiameter>0.34</wheelDiameter>
+      <!-- <torque>10</torque> -->
       <commandTopic>cmd_vel</commandTopic>
       <odometryTopic>odom</odometryTopic>
@@ -208,6 +263,6 @@
       <publishWheelJointState>false</publishWheelJointState>
       <rosDebugLevel>na</rosDebugLevel>
-      <wheelAcceleration>0</wheelAcceleration>
-      <wheelTorque>5</wheelTorque>
+      <wheelAcceleration>1</wheelAcceleration>
+      <wheelTorque>10</wheelTorque>
       <odometrySource>world</odometrySource>
       <publishTf>1</publishTf>
@@ -215,31 +270,32 @@
   </gazebo>
   <gazebo reference="hokuyo">
-    <sensor type="ray" name="head_hokuyo_sensor">
+    <material>Gazebo/FlatBlack</material>
+    <sensor type="ray" name="lds_lfcd_sensor">
       <pose>0 0 0 0 0 0</pose>
       <visualize>true</visualize>
-      <update_rate>40</update_rate>
+      <update_rate>5</update_rate>
       <ray>
         <scan>
           <horizontal>
-            <samples>720</samples>
+            <samples>360</samples>
             <resolution>1</resolution>
-            <min_angle>-1.570796</min_angle>
-            <max_angle>1.570796</max_angle>
+            <min_angle>0.0</min_angle>
+            <max_angle>6.28319</max_angle>
           </horizontal>
         </scan>
         <range>
-          <min>0.1</min>
-          <max>30.0</max>
-          <resolution>0.01</resolution>
+          <min>0.12</min>
+          <max>10</max>
+          <resolution>0.015</resolution>
         </range>
         <noise>
           <type>gaussian</type>
           <mean>0.0</mean>
-          <stddev>0.0</stddev>
+          <stddev>0.01</stddev>
         </noise>
       </ray>
-      <plugin name="gazebo_ros_head_hokuyo_controller" filename="libgazebo_ros_laser.so">
-        <topicName>/mybot/laser/scan</topicName>
-        <frameName>hokuyo</frameName>
+      <plugin name="gazebo_ros_lds_lfcd_controller" filename="libgazebo_ros_laser.so">
+        <topicName>scan</topicName>
+        <frameName>base_scan</frameName>
       </plugin>
     </sensor>
